File: hardware/dac.sch (KiCad schematic (older format))
At the start: 3 parts

Commit message: add hierarchical labels for dac outputs
Connections:
- net OUTH: now reaches U?.10 (VOUTH)
- net OUTF: now reaches U?.11 (VOUTF)
- net OUTD: now reaches U?.12 (VOUTD)
- net OUTB: now reaches U?.13 (VOUTB)
- net OUTA: now reaches U?.4 (VOUTA)
- net OUTC: now reaches U?.5 (VOUTC)
- net OUTE: now reaches U?.6 (VOUTE)
- net OUTG: now reaches U?.7 (VOUTG)
Changed lines of the file:
@@
 Text Label 6050 3550 2    50   ~ 0
 GND
+Text HLabel 4650 3650 0    50   Output ~ 0
+OUTA
+Text HLabel 6050 3650 2    50   Output ~ 0
+OUTB
+Text HLabel 4650 3750 0    50   Output ~ 0
+OUTC
+Text HLabel 6050 3750 2    50   Output ~ 0
+OUTD
+Text HLabel 4650 3850 0    50   Output ~ 0
+OUTE
+Text HLabel 6050 3850 2    50   Output ~ 0
+OUTF
+Text HLabel 4650 3950 0    50   Output ~ 0
+OUTG
+Text HLabel 6050 3950 2    50   Output ~ 0
+OUTH
 $EndSCHEMATC
